Commit message: Test and fix some bug, testing passed

File: src/rm2_description/urdf/common/mecanum_wheel.urdf.xacro (robot description, xacro)
@@ -85,5 +85,5 @@
         </link>
         <!--  joint  -->
-        <joint name="${prefix}_wheel_joint" type="revolute">
+        <joint name="${prefix}_wheel_joint" type="continuous">
             <axis xyz="0 1 0"/>
             <origin xyz="${wheel_x_offset} ${wheel_y_offset} ${wheel_offset_z}" rpy="0 0 0"/>

File: src/rm2_description/urdf/common/mecanum_wheel_14roller.urdf.xacro (robot description, xacro)
@@ -83,5 +83,5 @@
         </link>
         <!--  joint  -->
-        <joint name="${prefix}_wheel_joint" type="revolute">
+        <joint name="${prefix}_wheel_joint" type="continuous">
             <axis xyz="0 1 0"/>
             <origin xyz="${wheel_x_offset} ${wheel_y_offset} ${wheel_offset_z}" rpy="0 0 0"/>

File: src/rm2_description/urdf/common/omni_wheel.urdf.xacro (robot description, xacro)
@@ -70,5 +70,5 @@
         </link>
         <!--  joint  -->
-        <joint name="${prefix}_wheel_joint" type="revolute">
+        <joint name="${prefix}_wheel_joint" type="continuous">
             <axis xyz="0 1 0"/>
             <origin xyz="${wheel_x_offset} ${wheel_y_offset} ${wheel_offset_z}" rpy="0 0 ${rotation_degree}"/>

File: src/rm2_description/urdf/standard6/chassis.urdf.xacro (robot description, xacro)
@@ -31,12 +31,12 @@
                           max_effort="3.42" max_velocity="73"
         />
+        <xacro:omni_wheel prefix="left_back" connected_to="base_link"
+                          wheel_x_offset="${-chassis_radius/sqrt(2)}" wheel_y_offset="${chassis_radius/sqrt(2)}"
+                          wheel_z_offset="${wheel_offset_z}" rotation_degree="${-3*pi/4}" roller_type="${roller_type}"
+                          max_effort="3.42" max_velocity="73"
+        />
         <xacro:omni_wheel prefix="right_front" connected_to="base_link"
                           wheel_x_offset="${chassis_radius/sqrt(2)}" wheel_y_offset="${-chassis_radius/sqrt(2)}"
                           wheel_z_offset="${wheel_offset_z}" rotation_degree="${pi/4}" roller_type="${roller_type}"
-                          max_effort="3.42" max_velocity="73"
-        />
-        <xacro:omni_wheel prefix="left_back" connected_to="base_link"
-                          wheel_x_offset="${-chassis_radius/sqrt(2)}" wheel_y_offset="${chassis_radius/sqrt(2)}"
-                          wheel_z_offset="${wheel_offset_z}" rotation_degree="${-3*pi/4}" roller_type="${roller_type}"
                           max_effort="3.42" max_velocity="73"
         />
@@ -47,6 +47,6 @@
         />
         <xacro:wheel_transmission prefix="left_front" mechanical_reduction="13"/>
+        <xacro:wheel_transmission prefix="left_back" mechanical_reduction="13"/>
         <xacro:wheel_transmission prefix="right_front" mechanical_reduction="13"/>
-        <xacro:wheel_transmission prefix="left_back" mechanical_reduction="13"/>
         <xacro:wheel_transmission prefix="right_back" mechanical_reduction="13"/>
     </xacro:macro>

File: src/rm2_description/urdf/standard6/standard6.urdf.xacro (robot description, xacro)
@@ -51,5 +51,5 @@
             <state_interface name="effort"/>
         </joint>
-        <joint name="right_front_wheel_joint">
+        <joint name="left_back_wheel_joint">
             <command_interface name="effort"/>
             <state_interface name="position"/>
@@ -57,5 +57,5 @@
             <state_interface name="effort"/>
         </joint>
-        <joint name="left_back_wheel_joint">
+        <joint name="right_front_wheel_joint">
             <command_interface name="effort"/>
             <state_interface name="position"/>
@@ -69,4 +69,48 @@
             <state_interface name="effort"/>
         </joint>
+        <transmission name="left_front_wheel_trans">
+            <type>transmission_interface/SimpleTransmission</type>
+            <plugin>transmission_interface/SimpleTransmission</plugin>
+            <joint name="left_front_wheel_joint" role="actuated">
+                <mechanical_reduction>13</mechanical_reduction>
+                <offset>0.0</offset>
+            </joint>
+            <actuator name="left_front_wheel_motor" role="actuated">
+                <mechanical_reduction>1</mechanical_reduction>
+            </actuator>
+        </transmission>
+        <transmission name="left_back_wheel_trans">
+            <type>transmission_interface/SimpleTransmission</type>
+            <plugin>transmission_interface/SimpleTransmission</plugin>
+            <joint name="left_back_wheel_joint" role="actuated">
+                <mechanical_reduction>13</mechanical_reduction>
+                <offset>0.0</offset>
+            </joint>
+            <actuator name="left_back_wheel_motor" role="actuated">
+                <mechanical_reduction>1</mechanical_reduction>
+            </actuator>
+        </transmission>
+        <transmission name="right_front_wheel_trans">
+            <type>transmission_interface/SimpleTransmission</type>
+            <plugin>transmission_interface/SimpleTransmission</plugin>
+            <joint name="right_front_wheel_joint" role="actuated">
+                <mechanical_reduction>13</mechanical_reduction>
+                <offset>0.0</offset>
+            </joint>
+            <actuator name="right_front_wheel_motor" role="actuated">
+                <mechanical_reduction>1</mechanical_reduction>
+            </actuator>
+        </transmission>
+        <transmission name="right_back_wheel_trans">
+            <type>transmission_interface/SimpleTransmission</type>
+            <plugin>transmission_interface/SimpleTransmission</plugin>
+            <joint name="right_back_wheel_joint" role="actuated">
+                <mechanical_reduction>13</mechanical_reduction>
+                <offset>0.0</offset>
+            </joint>
+            <actuator name="right_back_wheel_motor" role="actuated">
+                <mechanical_reduction>1</mechanical_reduction>
+            </actuator>
+        </transmission>
         <!--Other joint wait to added-->
     </ros2_control>

File: src/rm2_ecat/rm2_ecat_ros/urdf/test.urdf.xacro (robot description, xacro)
@@ -28,5 +28,5 @@
       <joint name="test_joint" role="actuated">
         <hardwareInterface>rm2_ecat_ros/RmEcatHardwareInterface</hardwareInterface>
-        <mechanical_reduction>1</mechanical_reduction>    <!-- M3508 19.2032 -->
+        <mechanical_reduction>19.2032</mechanical_reduction>    <!-- M3508 19.2032 -->
         <offset>0.0</offset>
       </joint>
